File: pcb/fets.kicad_sch (KiCad schematic)
At the start: 49 parts, among them J10 Screw_Terminal_01x02, J11 Screw_Terminal_01x02, J12 Screw_Terminal_01x02, J13 Screw_Terminal_01x02, J14 Screw_Terminal_01x02, J7 Screw_Terminal_01x02, J8 Screw_Terminal_01x02, J9 Screw_Terminal_01x02, Q1 PJA3404A, Q10 PJA3404A, Q11 BC846, Q12 PJA3404A, Q13 MCAC011P03L-TP, Q14 BC846, Q15 BC846, Q16 MCAC011P03L-TP, Q2 BC846, Q3 BC846, Q4 PJA3404A, Q5 BC846, Q6 PJA3404A, Q7 BC846, Q8 PJA3404A, Q9 BC846

Commit message: pretty much everything on schem done, though need to add circuit protection stuff and break out remaining pins
Parts:
- renumbered J13 to J10, J7 to J11, J8 to J12, J9 to J13, J10 to J14, J11 to J15, J12 to J16, J14 to J9, Q2 to Q1, Q8 to Q10, Q10 to Q11, Q15 to Q13, Q16 to Q14, Q14 to Q15, Q13 to Q16, Q3 to Q2, Q5 to Q3, Q1 to Q4, Q4 to Q5, Q9 to Q8, Q11 to Q9, R18 to R29, R20 to R30, R23 to R31, R19 to R32, R21 to R33, R24 to R34, R37 to R35, R17 to R36, R22 to R37, R25 to R38, R38 to R39, R39 to R40, R26 to R41, R29 to R42, R32 to R43, R27 to R44, R30 to R45, R33 to R46, R28 to R47, R31 to R48, R34 to R49, R40 to R50, R41 to R51, R36 to R52, R35 to R53

Commit message: yay schematic pretty much good, though I'm going to have to redo some work to split it into multiple kicad projects so I can have multiple separate boards
Parts:
- Q14, Q16: footprint MCAC100N08YATP -> MCAC011P03L:MCAC100N08YATP
- R29, R30, R31, R32, R33, R34, R35, R36, R37, R38, R39, R40, R41, R42, R43, R44, R45, R46, R47, R48, R49, R50, R51, R52, R53: footprint (none) -> Resistor_SMD:R_0402_1005Metric
Changed lines of the file:
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@@
 			)
 		)
-		(property "Footprint" ""
+		(property "Footprint" "Resistor_SMD:R_0402_1005Metric"
 			(at 40.64 98.298 90)
 			(effects
@@
 			)
 		)
-		(property "Footprint" ""
+		(property "Footprint" "Resistor_SMD:R_0402_1005Metric"
 			(at 73.66 182.88 0)
 			(effects
@@
 			)
 		)
-		(property "Footprint" ""
+		(property "Footprint" "Resistor_SMD:R_0402_1005Metric"
 			(at 97.282 53.34 90)
 			(effects
@@
 			)
 		)
-		(property "Footprint" ""
+		(property "Footprint" "Resistor_SMD:R_0402_1005Metric"
 			(at 93.98 60.198 90)
 			(effects
@@
 			)
 		)
-		(property "Footprint" ""
+		(property "Footprint" "Resistor_SMD:R_0402_1005Metric"
 			(at 40.64 60.198 90)
 			(effects
@@
 			)
 		)
-		(property "Footprint" ""
+		(property "Footprint" "Resistor_SMD:R_0402_1005Metric"
 			(at 43.942 53.34 90)
 			(effects
@@
 			)
 		)
-		(property "Footprint" ""
+		(property "Footprint" "Resistor_SMD:R_0402_1005Metric"
 			(at 151.13 150.368 90)
 			(effects
@@
 			)
 		)
-		(property "Footprint" ""
+		(property "Footprint" "Resistor_SMD:R_0402_1005Metric"
 			(at 163.83 138.43 0)
 			(effects
@@
 			)
 		)
-		(property "Footprint" ""
+		(property "Footprint" "Resistor_SMD:R_0402_1005Metric"
 			(at 107.442 83.82 90)
 			(effects
@@
 			)
 		)
-		(property "Footprint" ""
+		(property "Footprint" "Resistor_SMD:R_0402_1005Metric"
 			(at 54.102 83.82 90)
 			(effects
@@
 			)
 		)
-		(property "Footprint" ""
+		(property "Footprint" "Resistor_SMD:R_0402_1005Metric"
 			(at 93.98 98.298 90)
 			(effects
@@
 			)
 		)
-		(property "Footprint" "MCAC100N08YATP"
+		(property "Footprint" "MCAC011P03L:MCAC100N08YATP"
 			(at 259.08 229.54 0)
 			(effects
@@
 			)
 		)
-		(property "Footprint" ""
+		(property "Footprint" "Resistor_SMD:R_0402_1005Metric"
 			(at 54.102 45.72 90)
 			(effects
@@
 			)
 		)
-		(property "Footprint" ""
+		(property "Footprint" "Resistor_SMD:R_0402_1005Metric"
 			(at 220.98 150.368 90)
 			(effects
@@
 			)
 		)
-		(property "Footprint" ""
+		(property "Footprint" "Resistor_SMD:R_0402_1005Metric"
 			(at 97.282 91.44 90)
 			(effects
@@
 			)
 		)
-		(property "Footprint" "MCAC100N08YATP"
+		(property "Footprint" "MCAC011P03L:MCAC100N08YATP"
 			(at 189.23 229.54 0)
 			(effects
@@
 			)
 		)
-		(property "Footprint" ""
+		(property "Footprint" "Resistor_SMD:R_0402_1005Metric"
 			(at 233.68 138.43 0)
 			(effects
@@
 			)
 		)
-		(property "Footprint" ""
+		(property "Footprint" "Resistor_SMD:R_0402_1005Metric"
 			(at 48.26 187.198 90)
 			(effects
@@
 			)
 		)
-		(property "Footprint" ""
+		(property "Footprint" "Resistor_SMD:R_0402_1005Metric"
 			(at 107.442 121.92 90)
 			(effects
@@
 			)
 		)
-		(property "Footprint" ""
+		(property "Footprint" "Resistor_SMD:R_0402_1005Metric"
 			(at 43.942 91.44 90)
 			(effects
@@
 			)
 		)
-		(property "Footprint" ""
+		(property "Footprint" "Resistor_SMD:R_0402_1005Metric"
 			(at 93.98 136.398 90)
 			(effects
@@
 			)
 		)
-		(property "Footprint" ""
+		(property "Footprint" "Resistor_SMD:R_0402_1005Metric"
 			(at 97.282 129.54 90)
 			(effects
@@
 			)
 		)
-		(property "Footprint" ""
+		(property "Footprint" "Resistor_SMD:R_0402_1005Metric"
 			(at 40.64 136.398 90)
 			(effects
@@
 			)
 		)
-		(property "Footprint" ""
+		(property "Footprint" "Resistor_SMD:R_0402_1005Metric"
 			(at 73.66 175.26 0)
 			(effects
@@
 			)
 		)
-		(property "Footprint" ""
+		(property "Footprint" "Resistor_SMD:R_0402_1005Metric"
 			(at 107.442 45.72 90)
 			(effects
@@
 			)
 		)
-		(property "Footprint" ""
+		(property "Footprint" "Resistor_SMD:R_0402_1005Metric"
 			(at 54.102 121.92 90)
 			(effects
@@
 			)
 		)
-		(property "Footprint" ""
+		(property "Footprint" "Resistor_SMD:R_0402_1005Metric"
 			(at 43.942 129.54 90)
 			(effects
