File: pcb/irisv2.kicad_sch (KiCad schematic)
At the start: 30 parts, among them J1 USB_C_Receptacle_USB2.0_16P, J2 USB_C_Receptacle_USB2.0_16P, J3 Screw_Terminal_01x02, U1 INA237, U2 MP4323GDE-Z

Commit message: fixed super minor issues
Parts:
- C8, C9: value 4.7uH -> 4.7uF
- J3: footprint (none) -> TerminalBlock_MetzConnect:TerminalBlock_MetzConnect_Type059_RT06302HBWC_1x02_P3.50mm_Horizontal
- U2: footprint QFN-12_MP4323_MNP -> MPM4323GDE:QFN-12_MP4323_MNP
Changed lines of the file:
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@@
 			)
 		)
-		(property "Footprint" "QFN-12_MP4323_MNP"
+		(property "Footprint" "MPM4323GDE:QFN-12_MP4323_MNP"
 			(at 170.18 81.28 0)
 			(effects
@@
 			)
 		)
-		(property "Value" "4.7uH"
+		(property "Value" "4.7uF"
 			(at 238.76 110.744 90)
 			(effects
@@
 			)
 		)
-		(property "Value" "4.7uH"
+		(property "Value" "4.7uF"
 			(at 238.76 122.936 90)
 			(effects
@@
 			)
 		)
-		(property "Footprint" ""
+		(property "Footprint" "TerminalBlock_MetzConnect:TerminalBlock_MetzConnect_Type059_RT06302HBWC_1x02_P3.50mm_Horizontal"
 			(at 30.48 34.29 0)
 			(effects

Commit message: tons of work on rf and mcu
Connections:
- net +5V renamed +5VP
- net scl renamed ina_scl
- net sda renamed ina_sda
Other:
- moved on the sheet: C1, C2

Commit message: sensors pretty much done (still need to add high g_
Parts:
- added C72: 47pF, symbol Device:C
- added C73: 2.2pF, symbol Device:C
- added C74: 18pF, symbol Device:C
- added C75: 22pF, symbol Device:C
- added C76: 7.5pF, symbol Device:C
- added C77, C79: 1.8pF, symbol Device:C
- added C78: 3.9pF, symbol Device:C
- added C95: 120pF, symbol Device:C
- added C96, C97, C98: 10uF, symbol Device:C
- added D5: D_TVS, symbol Device:D_TVS
- added D6: D_Schottky, symbol Device:D_Schottky
- added L16: 12nH, symbol Device:L
- added L17: 24nH, symbol Device:L
- added L18: 4.7nH, symbol Device:L
- added L19: 3.9nH, symbol Device:L
- added L20: 7.5nH, symbol Device:L
- added L21: 22nH, symbol Device:L
- added L22: 2.2uH, symbol Device:L
- added R14: 5, symbol Device:R
- added U11: TPS613222ADBV, Package_TO_SOT_SMD:SOT-23-5, symbol Regulator_Switching:TPS613222ADBV
- added V1: VSIN, symbol Simulation_SPICE:VSIN
Connections:
- net +3.3V: now also L22.1
- net GND renamed 0
- net 0: now also C72.1, C73.2, C76.2, C78.2, C79.2, C96.2, C97.2, C98.2, D5.1 (A1), L21.2, U11.2 (GND), V1.2
- new net: C75.2, C76.1, C77.1, L19.1
- new net: C77.2, C78.1, L19.2, L20.1
- new net: C75.1, L18.2
- new net: C95.1, R14.2
- new net: D6.2 (A), L22.2, R14.1, U11.1 (SW)
- new net: C73.1, C74.1, L17.2
- new net +5V: C95.2, C96.1, C97.1, C98.1, D6.1 (K), U11.4 (VOUT)
- new net lf_ant: C74.2, C79.1, D5.2 (A2), L20.2, L21.1
- new net lfi: L17.1
- new net lfo: L16.2, L18.1, V1.1
- new net vr_pa: C72.2, L16.1
Other:
- note added: "3.3v regulation"
- note added: "5v regulation"
- note removed: "power regulation"

Commit message: got fets figured out (finally), can integrated, a 5v regulator, sensors added - overall great progress!
Parts:
- R5: value R -> 0.015
- renumbered C72 to C1, C96 to C10, C97 to C11, C98 to C12, C1 to C13, C2 to C14, C4 to C15, C7 to C16, C5 to C17, C6 to C18, C3 to C19, C73 to C2, C10 to C20, C11 to C21, C8 to C22, C9 to C23, C74 to C3, C75 to C4, C76 to C5, C77 to C6, C78 to C7, C79 to C8, C95 to C9, D5 to D1, D1 to D2, D6 to D3, J3 to J1, J1 to J2, J2 to J3, L16 to L1, L17 to L2, L18 to L3, L19 to L4, L20 to L5, L21 to L6, L22 to L7, L1 to L8, R8 to R10, R6 to R11, R14 to R6, R10 to R8, U11 to U1, U1 to U2, U2 to U3
Other:
- added sheet fets (fets.kicad_sch)
- note removed: "todo determine shunt resistor value"

Commit message: pretty much everything on schem done, though need to add circuit protection stuff and break out remaining pins
Parts:
- removed C1: 47pF, symbol Device:C
- removed C2: 2.2pF, symbol Device:C
- removed C3: 18pF, symbol Device:C
- removed C4: 22pF, symbol Device:C
- removed C5: 7.5pF, symbol Device:C
- removed C6, C8: 1.8pF, symbol Device:C
- removed C7: 3.9pF, symbol Device:C
- removed D1: D_TVS, symbol Device:D_TVS
- removed L1: 12nH, symbol Device:L
- removed L2: 24nH, symbol Device:L
- removed L3: 4.7nH, symbol Device:L
- removed L4: 3.9nH, symbol Device:L
- removed L5: 7.5nH, symbol Device:L
- removed L6: 22nH, symbol Device:L
- removed V1: VSIN, symbol Simulation_SPICE:VSIN
- added D3: 3.3_GOOD, symbol Device:LED
- added D4: 5_GOOD, symbol Device:LED
- added R11: 580, symbol Device:R
- added R8: 240, symbol Device:R
- renumbered C9 to C1, C18 to C10, C19 to C11, C20 to C12, C21 to C13, C22 to C14, C23 to C15, C10 to C2, C11 to C3, C12 to C4, C13 to C5, C14 to C6, C15 to C7, C16 to C8, C17 to C9, D2 to D1, D3 to D2, L7 to L1, L8 to L2, R9 to R10, R10 to R12, R11 to R13, R8 to R9
Connections:
- net +3.3V: now also D3.2 (A)
- net +5V: now also D4.2 (A)
- net usb1_d+: no longer J3.A6 (D+), J3.B6 (D+)
- net usb1_d-: no longer J3.A7 (D-), J3.B7 (D-)
- net 0 renamed GND
- net GND: now also R11.1, R8.1
- new net: D4.1 (K), R11.2
- new net: D3.1 (K), R8.2
- new net usb2_d+: J3.A6 (D+), J3.B6 (D+)
- new net usb2_d-: J3.A7 (D-), J3.B7 (D-)
Other:
- note added: "green"
- note added: "power indication"
- note added: "yellow"
- note removed: "todo make my own symbol for this regulator"

Commit message: yay schematic pretty much good, though I'm going to have to redo some work to split it into multiple kicad projects so I can have multiple separate boards
Parts:
- C1, C11, C12, C13, C5, C7, C8: footprint (none) -> Capacitor_SMD:C_0603_1608Metric
- C10, C14, C15, C9: footprint (none) -> Capacitor_SMD:C_1210_3225Metric
- C2, C3, C4: footprint (none) -> Capacitor_SMD:C_1206_3216Metric
- C6: footprint (none) -> Capacitor_SMD:C_0402_1005Metric
- J2, J3: footprint (none) -> UJ20-C-H-G-SMT-1-P16-TR:SAMESKY_UJ20-C-H-G-SMT-1-P16-TR
- R1, R2, R3, R4: footprint (none) -> Resistor_SMD:R_0402_1005Metric
- R10, R11, R12, R13, R6, R8, R9: footprint (none) -> Resistor_SMD:R_0603_1608Metric
- R5: footprint (none) -> Resistor_SMD:R_2512_6332Metric
- R7: footprint (none) -> Resistor_SMD:R_0201_0603Metric
Connections:
- net GND: now also FB1.1, FB2.1, J2.A1 (GND), J2.A12 (GND), J2.B1 (GND), J2.B12 (GND), J3.A1 (GND), J3.A12 (GND), J3.B1 (GND), J3.B12 (GND)
Other:
- note added: "todo: split this into multiple kicad projects so it can actually be different boards"
Changed lines of the file:
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@@
 		)
 	)
+	(text "todo: split this into multiple kicad projects so it can actually be different boards"
+		(exclude_from_sim no)
+		(at 102.108 118.618 0)
+		(effects
+			(font
+				(size 1.27 1.27)
+			)
+		)
+	)
 	(text "5v regulation"
 		(exclude_from_sim no)
@@
 	)
 	(junction
+		(at 31.75 160.02)
+		(diameter 0)
+		(color 0 0 0 0)
+	)
+	(junction
 		(at 233.68 119.38)
 		(diameter 0)
@@
 	)
 	(junction
+		(at 31.75 102.87)
+		(diameter 0)
+		(color 0 0 0 0)
+	)
+	(junction
 		(at 243.84 119.38)
 		(diameter 0)
@@
 	(wire
 		(pts
+			(xy 31.75 102.87) (xy 31.75 104.14)
+		)
+		(stroke
+			(width 0)
+			(type default)
+		)
+	)
+	(wire
+		(pts
 			(xy 222.25 81.28) (xy 220.98 81.28)
 		)
@@
 		)
 	)
+	(wire
+		(pts
+			(xy 31.75 161.29) (xy 31.75 160.02)
+		)
+		(stroke
+			(width 0)
+			(type default)
+		)
+	)
 	(label "feedback"
 		(at 218.44 93.98 0)
@@
 			)
 		)
-		(property "Footprint" ""
+		(property "Footprint" "UJ20-C-H-G-SMT-1-P16-TR:SAMESKY_UJ20-C-H-G-SMT-1-P16-TR"
 			(at 35.56 78.74 0)
 			(effects
@@
 			)
 		)
-		(property "Footprint" ""
+		(property "Footprint" "Resistor_SMD:R_0603_1608Metric"
 			(at 172.72 123.698 90)
 			(effects
@@
 			)
 		)
-		(property "Footprint" ""
+		(property "Footprint" "UJ20-C-H-G-SMT-1-P16-TR:SAMESKY_UJ20-C-H-G-SMT-1-P16-TR"
 			(at 35.56 135.89 0)
 			(effects
@@
 			)
 		)
-		(property "Footprint" ""
+		(property "Footprint" "Resistor_SMD:R_0402_1005Metric"
 			(at 52.07 126.492 90)
 			(effects
@@
 			)
 		)
-		(property "Footprint" ""
+		(property "Footprint" "Capacitor_SMD:C_1206_3216Metric"
 			(at 126.0348 167.64 0)
 			(effects
@@
 			)
 		)
-		(property "Footprint" ""
+		(property "Footprint" "Capacitor_SMD:C_1210_3225Metric"
 			(at 203.2 121.6152 0)
 			(effects
@@
 			)
 		)
-		(property "Footprint" ""
+		(property "Footprint" "Resistor_SMD:R_0603_1608Metric"
 			(at 182.88 120.142 90)
 			(effects
@@
 			)
 		)
-		(property "Footprint" ""
+		(property "Footprint" "Capacitor_SMD:C_1210_3225Metric"
 			(at 210.82 114.6048 0)
 			(effects
@@
 			)
 		)
-		(property "Footprint" ""
+		(property "Footprint" "Resistor_SMD:R_0603_1608Metric"
 			(at 214.63 88.9 0)
 			(effects
@@
 			)
 		)
-		(property "Footprint" ""
+		(property "Footprint" "Capacitor_SMD:C_1206_3216Metric"
 			(at 120.9548 167.64 0)
 			(effects
@@
 			)
 		)
-		(property "Footprint" ""
+		(property "Footprint" "Capacitor_SMD:C_0603_1608Metric"
 			(at 224.79 120.3452 0)
 			(effects
@@
 			)
 		)
-		(property "Footprint" ""
+		(property "Footprint" "Resistor_SMD:R_0402_1005Metric"
 			(at 52.07 69.342 90)
 			(effects
@@
 			)
 		)
-		(property "Footprint" ""
+		(property "Footprint" "Capacitor_SMD:C_0603_1608Metric"
 			(at 213.0552 80.01 0)
 			(effects
@@
 			)
 		)
-		(property "Footprint" ""
+		(property "Footprint" "Capacitor_SMD:C_0402_1005Metric"
 			(at 129.54 91.1352 0)
 			(effects
@@
 			)
 		)
-		(property "Footprint" ""
+		(property "Footprint" "Capacitor_SMD:C_0603_1608Metric"
 			(at 110.49 145.0848 0)
 			(effects
@@
 			)
 		)
-		(property "Footprint" ""
+		(property "Footprint" "Resistor_SMD:R_0201_0603Metric"
 			(at 165.1 90.678 90)
 			(effects
@@
 			)
 		)
-		(property "Footprint" ""
+		(property "Footprint" "Capacitor_SMD:C_0603_1608Metric"
 			(at 186.69 117.1448 0)
 			(effects
@@
 			)
 		)
-		(property "Footprint" ""
+		(property "Footprint" "Capacitor_SMD:C_0603_1608Metric"
 			(at 166.37 93.98 0)
 			(effects
@@
 	)
 	(symbol
+		(lib_id "power:GND")
+		(at 31.75 161.29 0)
+		(unit 1)
+		(exclude_from_sim no)
+		(in_bom yes)
+		(on_board yes)
+		(dnp no)
+		(property "Reference" "#PWR0172"
+			(at 31.75 167.64 0)
+			(effects
+				(font
+					(size 1.27 1.27)
+				)
+				(hide yes)
+			)
+		)
+		(property "Value" "GND"
+			(at 35.306 163.576 0)
+			(effects
+				(font
+					(size 1.27 1.27)
+				)
+			)
+		)
+		(property "Footprint" ""
+			(at 31.75 161.29 0)
+			(effects
+				(font
+					(size 1.27 1.27)
+				)
+				(hide yes)
+			)
+		)
+		(property "Datasheet" ""
+			(at 31.75 161.29 0)
+			(effects
+				(font
+					(size 1.27 1.27)
+				)
+				(hide yes)
+			)
+		)
+		(property "Description" "Power symbol creates a global label with name \"GND\" , ground"
+			(at 31.75 161.29 0)
+			(effects
+				(font
+					(size 1.27 1.27)
+				)
+				(hide yes)
+			)
+		)
+		(pin "1"
+		)
+		(instances
+			(project "irisv2"
+				(path "/689e90bc-813a-4b0d-8c5b-8f2a305549f3"
+					(reference "#PWR0172")
+					(unit 1)
+				)
+			)
+		)
+	)
+	(symbol
 		(lib_id "Device:R")
 		(at 52.07 68.58 90)
@@
 			)
 		)
-		(property "Footprint" ""
+		(property "Footprint" "Resistor_SMD:R_0402_1005Metric"
 			(at 52.07 70.358 90)
 			(effects
@@
 			)
 		)
-		(property "Footprint" ""
+		(property "Footprint" "Resistor_SMD:R_0603_1608Metric"
 			(at 214.63 91.44 0)
 			(effects
@@
 			)
 		)
-		(property "Footprint" ""
+		(property "Footprint" "Resistor_SMD:R_2512_6332Metric"
 			(at 90.932 92.71 90)
 			(effects
@@
 			)
 		)
-		(property "Footprint" ""
+		(property "Footprint" "Resistor_SMD:R_0603_1608Metric"
 			(at 93.98 147.828 90)
 			(effects
@@
 			)
 		)
-		(property "Footprint" ""
+		(property "Footprint" "Resistor_SMD:R_0603_1608Metric"
 			(at 198.12 154.178 90)
 			(effects
@@
 			)
 		)
-		(property "Footprint" ""
+		(property "Footprint" "Capacitor_SMD:C_0603_1608Metric"
 			(at 137.16 84.1248 0)
 			(effects
@@
 	)
 	(symbol
+		(lib_id "power:GND")
+		(at 31.75 104.14 0)
+		(unit 1)
+		(exclude_from_sim no)
+		(in_bom yes)
+		(on_board yes)
+		(dnp no)
+		(property "Reference" "#PWR0171"
+			(at 31.75 110.49 0)
+			(effects
+				(font
+					(size 1.27 1.27)
+				)
+				(hide yes)
+			)
+		)
+		(property "Value" "GND"
+			(at 35.306 106.426 0)
+			(effects
+				(font
+					(size 1.27 1.27)
+				)
+			)
+		)
+		(property "Footprint" ""
+			(at 31.75 104.14 0)
+			(effects
+				(font
+					(size 1.27 1.27)
+				)
+				(hide yes)
+			)
+		)
+		(property "Datasheet" ""
+			(at 31.75 104.14 0)
+			(effects
+				(font
+					(size 1.27 1.27)
+				)
+				(hide yes)
+			)
+		)
+		(property "Description" "Power symbol creates a global label with name \"GND\" , ground"
+			(at 31.75 104.14 0)
+			(effects
+				(font
+					(size 1.27 1.27)
+				)
+				(hide yes)
+			)
+		)
+		(pin "1"
+		)
+		(instances
+			(project "irisv2"
+				(path "/689e90bc-813a-4b0d-8c5b-8f2a305549f3"
+					(reference "#PWR0171")
+					(unit 1)
+				)
+			)
+		)
+	)
+	(symbol
 		(lib_id "Device:R")
 		(at 168.91 152.4 90)
@@
 			)
 		)
-		(property "Footprint" ""
+		(property "Footprint" "Resistor_SMD:R_0603_1608Metric"
 			(at 168.91 154.178 90)
 			(effects
@@
 			)
 		)
-		(property "Footprint" ""
+		(property "Footprint" "Capacitor_SMD:C_1210_3225Metric"
 			(at 242.57 113.3348 0)
 			(effects
@@
 			)
 		)
-		(property "Footprint" ""
+		(property "Footprint" "Capacitor_SMD:C_1206_3216Metric"
 			(at 115.8748 167.64 0)
 			(effects
@@
 			)
 		)
-		(property "Footprint" ""
+		(property "Footprint" "Capacitor_SMD:C_1210_3225Metric"
 			(at 234.95 120.3452 0)
 			(effects
@@
 			)
 		)
-		(property "Footprint" ""
+		(property "Footprint" "Capacitor_SMD:C_0603_1608Metric"
 			(at 232.41 113.3348 0)
 			(effects
@@
 			)
 		)
-		(property "Footprint" ""
+		(property "Footprint" "Resistor_SMD:R_0402_1005Metric"
 			(at 52.07 127.508 90)
 			(effects
