File: pcb/sensors.kicad_sch (KiCad schematic)
At the start: 0 parts

Commit message: sensors pretty much done (still need to add high g_
Parts:
- added C82, C87, C91, C94: 1uF, symbol Device:C
- added C83, C84, C85, C86, C89, C90, C92, C93: 100nF, symbol Device:C
- added C88: 10uF, symbol Device:C_Small
- added U10: MMC5983MA, MMC5983MA_MEM, symbol mmc5983ma:MMC5983MA
- added U7, U8: ICM-45686, U_2p5X3X0p81_LGA14L_TDK, symbol icm45686:ICM-45686
- added U9: BMP581, BMP581, symbol BMP581:BMP581
Connections:
- new net: C88.1, U10.10 (CAP)
- new net +3.3V: C82.1, C83.1, C84.1, C85.1, C86.1, C87.1, C89.1, C90.1, C91.1, C92.1, C93.1, C94.1, U10.13 (VDDIO), U10.2 (VDD), U7.5 (VDDIO), U7.8 (VDD), U8.5 (VDDIO), U8.8 (VDD), U9.1 (VDDIO), U9.10 (VDD)
- new net GND: C82.2, C83.2, C84.2, C85.2, C86.2, C87.2, C88.2, C89.2, C90.2, C91.2, C92.2, C93.2, C94.2, U10.11 (GND), U10.9 (GND), U7.6 (GND), U8.6 (GND), U9.3 (VSS_1), U9.8 (VSS_2), U9.9 (VSS_3)
- new net bmp_cs: U9.6 (CSB)
- new net bmp_int: U9.7 (INT)
- new net bmp_miso: U9.5 (SDO)
- new net bmp_mosi: U9.4 (SDI)
- new net bmp_sck: U9.2 (SCK)
- new net icm1_cs: U7.12 (AP_CS)
- new net icm1_miso: U7.1 (AP_SDO/AP_AD0)
- new net icm1_mosi: U7.14 (AP_SDA/AP_SDIO/AP_SDI)
- new net icm1_sck: U7.13 (AP_SCL/AP_SCLK)
- new net icm2_cs: U8.12 (AP_CS)
- new net icm2_miso: U8.1 (AP_SDO/AP_AD0)
- new net icm2_mosi: U8.14 (AP_SDA/AP_SDIO/AP_SDI)
- new net icm2_sck: U8.13 (AP_SCL/AP_SCLK)
- new net icm_fsync: U7.9 (INT2/FSYNC/CLKIN), U8.9 (INT2/FSYNC/CLKIN)
- new net imu1_int: U7.4 (INT1/INT)
- new net imu2_int: U8.4 (INT1/INT)
- new net mag_cs: U10.4 (SPI_CS)
- new net mag_int: U10.15 (INT)
- new net mag_miso: U10.5 (SPI_SDO)
- new net mag_mosi: U10.16 (SDA/SPI_SDI)
- new net mag_sck: U10.1 (SCL/SPI_SCK)
- no-connect marks 0 -> 16
Other:
- note added: "barometer"
- note added: "barometer decoupling"
- note added: "imu 1"
- note added: "imu 1 decoupling"
- note added: "imu 2"
- note added: "imu 2 decoupling"
- note added: "magnetometer"
- note added: "magnetometer decoupling"

Commit message: got fets figured out (finally), can integrated, a 5v regulator, sensors added - overall great progress!
Parts:
- renumbered C88 to C56, C92 to C57, C93 to C58, C84 to C59, C85 to C60, C94 to C61, C83 to C62, C86 to C63, C82 to C64, C87 to C65, C89 to C66, C90 to C67, C91 to C68, U10 to U5, U7 to U6, U8 to U7, U9 to U8
Other:
- moved on the sheet: C66, C67, C68, U8

Commit message: pretty much everything on schem done, though need to add circuit protection stuff and break out remaining pins
Parts:
- added AC1: H3LIS331DLTR, LIS3DHTR, symbol H3LIS331DLTR:H3LIS331DLTR
- added C67, C68: 100nF, symbol Device:C
- added C69, C70: 10uF, symbol Device:C
- renumbered C56 to C54, C57 to C55, C58 to C56, C59 to C57, C60 to C58, C61 to C59, C62 to C60, C63 to C61, C64 to C62, C65 to C63, C66 to C64, C67 to C65, C68 to C66
Connections:
- net +3.3V: now also AC1.1 (VDD_IO), AC1.14 (VDD), C67.1, C68.1, C69.1, C70.1
- net GND: now also AC1.12 (GND_2), AC1.13 (GND_3), AC1.16 (GND_4), AC1.5 (GND_1), C67.2, C68.2, C69.2, C70.2
- net imu1_int renamed icm1_int
- net imu2_int renamed icm2_int
- new net hig_cs: AC1.8 (CS)
- new net hig_miso: AC1.7 (SDO_SA0)
- new net hig_mosi: AC1.6 (SDA_SDI_SDO)
- new net hig_sck: AC1.4 (SCL_SPC)
- new net highg_int: AC1.11 (INT1)
- no-connect marks 16 -> 21
Other:
- note added: "high g accel decoupling"
- note added: "high g accelerometer"
- moved on the sheet: C64, C65, C66, U8

Commit message: yay schematic pretty much good, though I'm going to have to redo some work to split it into multiple kicad projects so I can have multiple separate boards
Parts:
- AC1: footprint LIS3DHTR -> H3LIS331DLTR:LIS3DHTR
- C54, C59, C62, C63, C66, C69, C70: footprint (none) -> Capacitor_SMD:C_0603_1608Metric
- C55, C56, C57, C58, C60, C61, C64, C65, C67, C68: footprint (none) -> Capacitor_SMD:C_0402_1005Metric
- U5: footprint MMC5983MA_MEM -> mmc5983ma:MMC5983MA_MEM
- U6, U7: footprint U_2p5X3X0p81_LGA14L_TDK -> icm45686:U_2p5X3X0p81_LGA14L_TDK
- U8: footprint BMP581 -> BMP581:BMP581
Changed lines of the file:
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@@
 			)
 		)
-		(property "Footprint" ""
+		(property "Footprint" "Capacitor_SMD:C_0402_1005Metric"
 			(at 248.6152 115.57 0)
 			(effects
@@
 			)
 		)
-		(property "Footprint" ""
+		(property "Footprint" "Capacitor_SMD:C_0402_1005Metric"
 			(at 121.6152 156.21 0)
 			(effects
@@
 			)
 		)
-		(property "Footprint" ""
+		(property "Footprint" "Capacitor_SMD:C_0402_1005Metric"
 			(at 138.1252 95.25 0)
 			(effects
@@
 			)
 		)
-		(property "Footprint" "U_2p5X3X0p81_LGA14L_TDK"
+		(property "Footprint" "icm45686:U_2p5X3X0p81_LGA14L_TDK"
 			(at 29.21 90.17 0)
 			(effects
@@
 			)
 		)
-		(property "Footprint" ""
+		(property "Footprint" "Capacitor_SMD:C_0603_1608Metric"
 			(at 134.3152 156.21 0)
 			(effects
@@
 			)
 		)
-		(property "Footprint" ""
+		(property "Footprint" "Capacitor_SMD:C_0402_1005Metric"
 			(at 202.8952 80.01 0)
 			(effects
@@
 			)
 		)
-		(property "Footprint" "BMP581"
+		(property "Footprint" "BMP581:BMP581"
 			(at 226.06 125.4 0)
 			(effects
@@
 			)
 		)
-		(property "Footprint" ""
+		(property "Footprint" "Capacitor_SMD:C_0603_1608Metric"
 			(at 63.5 170.18 0)
 			(effects
@@
 			)
 		)
-		(property "Footprint" ""
+		(property "Footprint" "Capacitor_SMD:C_0402_1005Metric"
 			(at 108.9152 156.21 0)
 			(effects
@@
 			)
 		)
-		(property "Footprint" "LIS3DHTR"
+		(property "Footprint" "H3LIS331DLTR:LIS3DHTR"
 			(at 228.6 202.87 0)
 			(effects
@@
 			)
 		)
-		(property "Footprint" "U_2p5X3X0p81_LGA14L_TDK"
+		(property "Footprint" "icm45686:U_2p5X3X0p81_LGA14L_TDK"
 			(at 29.21 35.56 0)
 			(effects
@@
 			)
 		)
-		(property "Footprint" ""
+		(property "Footprint" "Capacitor_SMD:C_0402_1005Metric"
 			(at 125.4252 40.64 0)
 			(effects
@@
 			)
 		)
-		(property "Footprint" ""
+		(property "Footprint" "Capacitor_SMD:C_0402_1005Metric"
 			(at 125.4252 95.25 0)
 			(effects
@@
 			)
 		)
-		(property "Footprint" ""
+		(property "Footprint" "Capacitor_SMD:C_0402_1005Metric"
 			(at 215.5952 80.01 0)
 			(effects
@@
 			)
 		)
-		(property "Footprint" ""
+		(property "Footprint" "Capacitor_SMD:C_0603_1608Metric"
 			(at 261.3152 115.57 0)
 			(effects
@@
 			)
 		)
-		(property "Footprint" "MMC5983MA_MEM"
+		(property "Footprint" "mmc5983ma:MMC5983MA_MEM"
 			(at 27.94 147.32 0)
 			(effects
@@
 			)
 		)
-		(property "Footprint" ""
+		(property "Footprint" "Capacitor_SMD:C_0603_1608Metric"
 			(at 150.8252 95.25 0)
 			(effects
@@
 			)
 		)
-		(property "Footprint" ""
+		(property "Footprint" "Capacitor_SMD:C_0402_1005Metric"
 			(at 138.1252 40.64 0)
 			(effects
@@
 			)
 		)
-		(property "Footprint" ""
+		(property "Footprint" "Capacitor_SMD:C_0603_1608Metric"
 			(at 150.8252 40.64 0)
 			(effects
@@
 			)
 		)
-		(property "Footprint" ""
+		(property "Footprint" "Capacitor_SMD:C_0603_1608Metric"
 			(at 228.2952 80.01 0)
 			(effects
@@
 			)
 		)
-		(property "Footprint" ""
+		(property "Footprint" "Capacitor_SMD:C_0603_1608Metric"
 			(at 272.7452 115.57 0)
 			(effects
@@
 			)
 		)
-		(property "Footprint" ""
+		(property "Footprint" "Capacitor_SMD:C_0402_1005Metric"
 			(at 235.9152 115.57 0)
 			(effects
